File: Aktorik/Platine/Carolo_schaltplan.brd (EAGLE design)
At the start: 160 x 100 mm, 48 parts, among them IC1 TPS77301, IC2(SERVO) 74LVC1G157

Commit message: Board angefangen
Parts:
- removed 12V, BATTERIE, X6, X8: (no value), con-wago-508:W237-132
- removed X5, X7: (no value), con-wago-508:W237-133
- added U$1, U$2: XT60, XT60:XT60
- added X17, X18, X19: (no value), con-phoenix-254:12POL254
- X1: device con-wago-508:W237-12P -> con-phoenix-254:3POL254
- X10, X9: device con-wago-508:W237-12P -> con-phoenix-254:8POL254
- X11, X3, X4: device con-wago-508:W237-12P -> con-phoenix-254:12POL254
- X12: device con-wago-508:W237-8P -> con-phoenix-254:12POL254
- X13: device con-wago-508:W237-8P -> con-phoenix-254:5POL254
- X2: device con-wago-508:W237-12P -> con-phoenix-254:2POL254
- moved X12 514.3 mm to (384.9, -59.2), turned to 90 degrees
- moved X4 500.3 mm to (385.2, 5.04), turned to 90 degrees
- moved X13 471.6 mm to (384.5, -82.2), turned to 90 degrees
- moved X16 467.6 mm to (365.6, -12.2), turned to 270 degrees
- moved X11 454.6 mm to (385.2, -26.7), turned to 90 degrees
- moved X3 433.8 mm to (385.2, 36.8), turned to 90 degrees
- moved STARTSCHALTER 332.1 mm to (155.7, -29.2), turned to 90 degrees
- moved C2 321.7 mm to (142.0, -31.0), turned to 270 degrees
- moved C1 319.2 mm to (146.4, -31.4), turned to 270 degrees
- moved C3 303.7 mm to (142.2, 21.6), turned to 270 degrees
- moved L1 298.4 mm to (142.2, -11.4), turned to 180 degrees
- moved IC1 294.0 mm to (154.4, 4.45), turned to 180 degrees
- moved R1 286.9 mm to (160.0, 0.00), turned to 270 degrees
- moved R2 284.6 mm to (152.4, 17.8), turned to 270 degrees
- moved D1 279.6 mm to (156.2, -15.7), turned to 270 degrees
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Connections:
- removed net 5V: B1.VIN, C4.2, C6.1, C7.1, D2.C, IC2(SERVO).5, L1.1, MOTOR(FERNBEDIENUNG).3, R4.1, R8.2, SERVO.2, X1.1, X1.10, X1.11, X1.12, X1.2, X1.3, X1.4, X1.5, X1.6, X1.7, X1.8, X1.9, X15.2, X16.1, X2.1, X2.10, X2.11, X2.12, X2.2, X2.3, X2.4, X2.5, X2.6, X2.7, X2.8, X2.9
- removed net N$1 (its old number): 12V.2, C1.1, C2.1, D1.C, IC1.8, R1.2
- removed net N$10: B1.A1, X9.2
- new net N$2: C1.1, C2.1, D1.C, IC1.8, R1.2, U$2.+
- new net N$55: B1.A1, X17.11
- new net N$8: B1.VIN, C4.2, C6.1, C7.1, D2.C, IC2(SERVO).5, L1.1, MOTOR(FERNBEDIENUNG).3, R4.1, R8.2, SERVO.2, X15.2, X16.1, X3.1, X3.10, X3.11, X3.12, X3.2, X3.3, X3.4, X3.5, X3.6, X3.7, X3.8, X3.9, X4.1, X4.10, X4.11, X4.12, X4.2, X4.3, X4.4, X4.5, X4.6, X4.7, X4.8, X4.9
- net 3,3VARDUINO: now also X2.1, X2.2; no longer X6.1, X6.2
- net 5VARDUINO: now also X1.1, X1.2, X1.3; no longer X7.1, X7.2, X7.3
- net D22: now also X18.12; no longer X10.1
- net D24: now also X18.10; no longer X10.3
- net D26: now also X18.8; no longer X10.5
- net D28: now also X19.12; no longer X10.7
- net D30: now also X19.10; no longer X10.9
- net D32: now also X19.8; no longer X10.11
- net D34: now also X18.6; no longer X11.1
- net D36: now also X18.4; no longer X11.3
- net D38: now also X18.2; no longer X11.5
- net GND: now also U$2.-; no longer 12V.1, BATTERIE.1
- net N$11: now also U$1.+; no longer BATTERIE.2
- net N$12: now also X10.1, X10.2, X10.3, X10.4, X10.5, X10.6, X10.7, X10.8; no longer X12.1, X12.2, X12.3, X12.4, X12.5, X12.7, X12.8
- net N$18: now also X17.10; no longer X9.3
- net N$19: now also X17.9; no longer X9.4
- net N$20: now also X17.8; no longer X9.5
- net N$21: now also X17.7; no longer X9.6
- net N$22: now also X17.6; no longer X9.7
- net N$23: now also X17.5; no longer X9.8
- net N$24: now also X17.4; no longer X9.9
- net N$25: now also X17.3; no longer X9.10
- net N$26: now also X17.2; no longer X9.11
- net N$27: now also X17.1; no longer X9.12
- net N$28: now also X18.11; no longer X10.2
- net N$29: now also X9.1, X9.2, X9.3, X9.4, X9.5, X9.6, X9.7, X9.8; no longer X13.1, X13.3, X13.5, X13.6, X13.7, X13.8
- net N$30: now also X18.9; no longer X10.4
- net N$31: now also X18.7; no longer X10.6
- net N$32: now also X19.11; no longer X10.8
- net N$33: now also X19.9; no longer X10.10
- net N$34: now also X19.7; no longer X10.12
- net N$35: now also X18.5; no longer X11.2
- net N$36: now also X18.3; no longer X11.4
- net N$6: now also X11.1, X11.10, X11.11, X11.12, X11.2, X11.3, X11.4, X11.5, X11.6, X11.7, X11.8, X11.9, X12.1, X12.10, X12.11, X12.12, X12.2, X12.3, X12.4, X12.5, X12.6, X12.7, X12.8, X12.9, X13.1, X13.2, X13.3, X13.4, X13.5; no longer X3.1, X3.10, X3.11, X3.12, X3.2, X3.3, X3.4, X3.5, X3.6, X3.7, X3.8, X3.9, X4.1, X4.10, X4.11, X4.12, X4.2, X4.3, X4.4, X4.5, X4.6, X4.7, X4.8, X4.9, X5.1, X5.2, X5.3, X8.1, X8.2
- net N$9: now also X17.12; no longer X9.1
- net PIN1: now also X19.1; no longer X11.12
- net PIN10: now also X19.5; no longer X11.8
- net PIN18: now also X19.6; no longer X11.7
- net PIN19: now also X18.1; no longer X11.6
- net PIN2: now also X19.2; no longer X11.11
- net PIN3: now also X19.3; no longer X11.10
- net PIN9: now also X19.4; no longer X11.9
Routing:
- net GND: track 0.00 -> 283.2 mm
- net N$8: track 0.00 -> 238.8 mm
- net N$3: track 0.00 -> 168.9 mm
- net SL: track 0.00 -> 59.7 mm
- net N$43: track 0.00 -> 56.0 mm
- net N$40: track 0.00 -> 41.0 mm
- net N$12: track 0.00 -> 38.1 mm
- net N$1: track 0.00 -> 36.8 mm
- net N$29: track 0.00 -> 33.0 mm
- net N$52: track 0.00 -> 26.7 mm
- net TIEFPASS: track 0.00 -> 24.1 mm
- net N$51: track 0.00 -> 22.9 mm
- net N$2: track 0.00 -> 16.5 mm
- net 5VARDUINO: track 0.00 -> 15.4 mm
- net N$7: track 0.00 -> 14.0 mm
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Other:
- board size 160 x 100 mm -> 107 x 150 mm

Commit message: neuer Status
Parts:
- moved SV1 30.5 mm to (64.8, 97.8)
- moved R6 25.6 mm to (80.0, 99.1), turned to 0 degrees
- moved X19 3.59 mm to (59.7, 47.0)
- moved X18 1.27 mm to (98.2, 81.5)
- moved IC2(SERVO) 1.27 mm to (121.6, 83.9)
Routing:
- net TIEFPASS_PWM: track 0.00 -> 106.7 mm
- net N$38: track 0.00 -> 101.5 mm
- net N$37: track 0.00 -> 6.35 mm
