File: Aktorik/Platine/Carolo_schaltplan.sch (EAGLE design)
At the start: 47 parts, among them IC1 TPS77301, IC2(SERVO) 74LVC1G157

Commit message: Board angefangen
Parts:
- removed 12V, BATTERIE, X6, X8: (no value), con-wago-508:W237-02P
- removed X5, X7: (no value), con-wago-508:W237-03P
- added SV1: (no value), con-harting-ml:ML6
- added U$1, U$2: XT60, XT60:XT60
- added X17, X18, X19: (no value), con-phoenix-254:MPT12
- X1: device con-wago-508:W237-12P -> con-phoenix-254:MPT3
- X10, X9: device con-wago-508:W237-12P -> con-phoenix-254:MPT8
- X11, X3, X4: device con-wago-508:W237-12P -> con-phoenix-254:MPT12
- X12: device con-wago-508:W237-08P -> con-phoenix-254:MPT12
- X13: device con-wago-508:W237-08P -> con-phoenix-254:MPT5
- X2: device con-wago-508:W237-12P -> con-phoenix-254:MPT2
Connections:
- removed net 5V: B1.VIN, C4.2, C6.1, C7.1, D2.C, IC2(SERVO)P.VCC, L1.1, MOTOR(FERNBEDIENUNG)-3.S, R4.1, R8.2, SERVO-2.S, X1-1.KL, X1-10.KL, X1-11.KL, X1-12.KL, X1-2.KL, X1-3.KL, X1-4.KL, X1-5.KL, X1-6.KL, X1-7.KL, X1-8.KL, X1-9.KL, X15-2.KL, X16-1.KL, X2-1.KL, X2-10.KL, X2-11.KL, X2-12.KL, X2-2.KL, X2-3.KL, X2-4.KL, X2-5.KL, X2-6.KL, X2-7.KL, X2-8.KL, X2-9.KL
- removed net N$1 (its old number): 12V-2.KL, C1.1, C2.1, D1.C, IC1.VIN, R1.2
- removed net N$10: B1.A1, X9-2.KL
- removed net N$43: MOTOR(FERNBEDIENUNG)-1.S, R6.1
- new net N$2: C1.1, C2.1, D1.C, IC1.VIN, R1.2, U$2.VCC
- new net N$37: R6.1, SV1.6
- new net N$38: MOTOR(FERNBEDIENUNG)-1.S, SV1.1, SV1.3, SV1.5
- new net N$55: B1.A1, X17-11.1
- new net N$8: B1.VIN, C4.2, C6.1, C7.1, D2.C, IC2(SERVO)P.VCC, L1.1, MOTOR(FERNBEDIENUNG)-3.S, R4.1, R8.2, SERVO-2.S, X15-2.KL, X16-1.KL, X3-1.1, X3-10.1, X3-11.1, X3-12.1, X3-2.1, X3-3.1, X3-4.1, X3-5.1, X3-6.1, X3-7.1, X3-8.1, X3-9.1, X4-1.1, X4-10.1, X4-11.1, X4-12.1, X4-2.1, X4-3.1, X4-4.1, X4-5.1, X4-6.1, X4-7.1, X4-8.1, X4-9.1
- new net TIEFPASS_OPT: B1.39, SV1.4
- new net TIEFPASS_PWM: B1.4, SV1.2
- net 3,3VARDUINO: now also X2-1.1, X2-2.1; no longer X6-1.KL, X6-2.KL
- net 5VARDUINO: now also X1-1.1, X1-2.1, X1-3.1; no longer X7-1.KL, X7-2.KL, X7-3.KL
- net D22: now also X18-12.1; no longer X10-1.KL
- net D24: now also X18-10.1; no longer X10-3.KL
- net D26: now also X18-8.1; no longer X10-5.KL
- net D28: now also X19-12.1; no longer X10-7.KL
- net D30: now also X19-10.1; no longer X10-9.KL
- net D32: now also X19-8.1; no longer X10-11.KL
- net D34: now also X18-6.1; no longer X11-1.KL
- net D36: now also X18-4.1; no longer X11-3.KL
- net D38: now also X18-2.1; no longer X11-5.KL
- net GND: now also U$2.GND; no longer 12V-1.KL, BATTERIE-1.KL
- net N$11: now also U$1.VCC; no longer BATTERIE-2.KL
- net N$12: now also X10-1.1, X10-2.1, X10-3.1, X10-4.1, X10-5.1, X10-6.1, X10-7.1, X10-8.1; no longer X12-1.KL, X12-2.KL, X12-3.KL, X12-4.KL, X12-5.KL, X12-7.KL, X12-8.KL
- net N$18: now also X17-10.1; no longer X9-3.KL
- net N$19: now also X17-9.1; no longer X9-4.KL
- net N$20: now also X17-8.1; no longer X9-5.KL
- net N$21: now also X17-7.1; no longer X9-6.KL
- net N$22: now also X17-6.1; no longer X9-7.KL
- net N$23: now also X17-5.1; no longer X9-8.KL
- net N$24: now also X17-4.1; no longer X9-9.KL
- net N$25: now also X17-3.1; no longer X9-10.KL
- net N$26: now also X17-2.1; no longer X9-11.KL
- net N$27: now also X17-1.1; no longer X9-12.KL
- net N$28: now also X18-11.1; no longer X10-2.KL
- net N$29: now also X9-1.1, X9-2.1, X9-3.1, X9-4.1, X9-5.1, X9-6.1, X9-7.1, X9-8.1; no longer X13-1.KL, X13-3.KL, X13-5.KL, X13-6.KL, X13-7.KL, X13-8.KL
- net N$30: now also X18-9.1; no longer X10-4.KL
- net N$31: now also X18-7.1; no longer X10-6.KL
- net N$32: now also X19-11.1; no longer X10-8.KL
- net N$33: now also X19-9.1; no longer X10-10.KL
- net N$34: now also X19-7.1; no longer X10-12.KL
- net N$35: now also X18-5.1; no longer X11-2.KL
- net N$36: now also X18-3.1; no longer X11-4.KL
- net N$6: now also X11-1.1, X11-10.1, X11-11.1, X11-12.1, X11-2.1, X11-3.1, X11-4.1, X11-5.1, X11-6.1, X11-7.1, X11-8.1, X11-9.1, X12-1.1, X12-10.1, X12-11.1, X12-12.1, X12-2.1, X12-3.1, X12-4.1, X12-5.1, X12-6.1, X12-7.1, X12-8.1, X12-9.1, X13-1.1, X13-2.1, X13-3.1, X13-4.1, X13-5.1; no longer X3-1.KL, X3-10.KL, X3-11.KL, X3-12.KL, X3-2.KL, X3-3.KL, X3-4.KL, X3-5.KL, X3-6.KL, X3-7.KL, X3-8.KL, X3-9.KL, X4-1.KL, X4-10.KL, X4-11.KL, X4-12.KL, X4-2.KL, X4-3.KL, X4-4.KL, X4-5.KL, X4-6.KL, X4-7.KL, X4-8.KL, X4-9.KL, X5-1.KL, X5-2.KL, X5-3.KL, X8-1.KL, X8-2.KL
- net N$9: now also X17-12.1; no longer X9-1.KL
- net PIN1: now also X19-1.1; no longer X11-12.KL
- net PIN10: now also X19-5.1; no longer X11-8.KL
- net PIN18: now also X19-6.1; no longer X11-7.KL
- net PIN19: now also X18-1.1; no longer X11-6.KL
- net PIN2: now also X19-2.1; no longer X11-11.KL
- net PIN3: now also X19-3.1; no longer X11-10.KL
- net PIN9: now also X19-4.1; no longer X11-9.KL
Other:
- moved on the sheet: R6

Commit message: new Upload
Parts:
- removed X10: (no value), con-phoenix-254:MPT8
- removed X11, X12, X3, X4: (no value), con-phoenix-254:MPT12
- removed X13: (no value), con-phoenix-254:MPT5
- removed X16: (no value), con-wago-500:W237-102
Connections:
- removed net D28: B1.28, X19-12.1
- removed net D30: B1.30, X19-10.1
- removed net D32: B1.32, X19-8.1
- removed net D34: B1.34, X18-6.1
- removed net D36: B1.36, X18-4.1
- removed net D38: B1.38, X18-2.1
- removed net D40: B1.40
- removed net D42: B1.42
- removed net D44: B1.44
- removed net N$45: B1.50/MISO, X14-2.KL
- removed net N$6: X11-1.1, X11-10.1, X11-11.1, X11-12.1, X11-2.1, X11-3.1, X11-4.1, X11-5.1, X11-6.1, X11-7.1, X11-8.1, X11-9.1, X12-1.1, X12-10.1, X12-11.1, X12-12.1, X12-2.1, X12-3.1, X12-4.1, X12-5.1, X12-6.1, X12-7.1, X12-8.1, X12-9.1, X13-1.1, X13-2.1, X13-3.1, X13-4.1, X13-5.1, X16-2.KL
- removed net TIEFPASS_PWM: B1.4, SV1.2
- new net N$5: B1.27, X18-11.1
- new net SDA: B1.20(SDA), X19-10.1, X19-11.1, X19-12.1, X19-8.1, X19-9.1
- new net TIEFPASS_DIGITAL: B1.22, SV1.2
- net 5VARDUINO: now also MOTOR(FERNBEDIENUNG)-3.S, SERVO-2.S
- net D22: now also B1.25; no longer B1.22
- net D24: now also B1.29; no longer B1.24
- net D26: now also B1.33; no longer B1.26
- net GND: now also MOTOR(FERNBEDIENUNG)-2.S, MOTOR-2.S, U$1.GND
- net N$12: now also B1.31, X18-9.1; no longer B1.20(SDA), X10-1.1, X10-2.1, X10-3.1, X10-4.1, X10-5.1, X10-6.1, X10-7.1, X10-8.1
- net N$14: now also B1.5; no longer B1.12
- net N$17: now also B1.6, MOTOR-1.S; no longer B1.11
- net N$18: now also B1.A2
- net N$20: now also B1.A4
- net N$23: now also B1.A7
- net N$24: now also B1.A8
- net N$25: now also B1.A9
- net N$28: now also B1.35, X18-7.1; no longer B1.23, X18-11.1
- net N$30: now also B1.37, X18-6.1; no longer B1.25, X18-9.1
- net N$31: now also B1.39, X18-5.1; no longer B1.27, X18-7.1
- net N$32: now also B1.41, X18-4.1; no longer X19-11.1
- net N$33: now also B1.43, X18-3.1; no longer X19-9.1
- net N$34: now also B1.45, X18-2.1; no longer X19-7.1
- net N$35: now also B1.47, X18-1.1; no longer X18-5.1
- net N$36: now also B1.52/SCK, X14-2.KL; no longer X18-3.1
- net N$42: now also X14-1.KL
- net N$44: now also B1.50/MISO; no longer B1.52/SCK
- net N$8: no longer MOTOR(FERNBEDIENUNG)-3.S, SERVO-2.S, X16-1.KL, X3-1.1, X3-10.1, X3-11.1, X3-12.1, X3-2.1, X3-3.1, X3-4.1, X3-5.1, X3-6.1, X3-7.1, X3-8.1, X3-9.1, X4-1.1, X4-10.1, X4-11.1, X4-12.1, X4-2.1, X4-3.1, X4-4.1, X4-5.1, X4-6.1, X4-7.1, X4-8.1, X4-9.1
- net N$9: now also B1.A0
- net PIN1: now also X19-5.1; no longer X19-1.1
- net PIN10: now also X19-1.1; no longer X19-5.1
- net PIN19: now also X19-7.1; no longer X18-1.1
- net PIN2: now also X19-4.1; no longer X19-2.1
- net PIN9: now also X19-2.1; no longer X19-4.1
- net SL: now also B1.49; no longer B1.46
- net TIEFPASS_OPT: now also B1.4; no longer B1.39
Other:
- note removed: "5V"
- note removed: "GND"
- moved on the sheet: X1-1, X1-2, X1-3, X18-1, X18-2, X18-3, X18-4, X18-5, X18-6, X19-10, X19-11, X19-12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
